Commit message: LiDARを搭載する前提でURDF・地図等を追加

File: tsuten_description/urdf/tsuten.urdf.xacro (robot description, xacro)
@@ -1,4 +1,5 @@
 <?xml version="1.0" encoding="UTF-8"?>
 <robot name="tsuten" xmlns:xacro="http://ros.org/wiki/xacro">
+  <xacro:include filename="$(find tsuten_description)/urdf/lidar.urdf.xacro" />
   <xacro:include filename="$(find tsuten_description)/urdf/material.urdf.xacro" />
   <xacro:include filename="$(find tsuten_description)/urdf/wheel.urdf.xacro" />
@@ -68,4 +69,7 @@
     <origin xyz="325.1e-3 -359.1e-3 -242.3e-3" rpy="${radians(-45)} ${radians(-90)} 0" />
   </xacro:wheel>
+  <xacro:lidar parent="body_link">
+    <origin xyz="-30.69e-3 283.7e-3 -164.8e-3" rpy="0 0 ${radians(90)}" />
+  </xacro:lidar>
   <gazebo reference="body_link">
     <material>

File: tsuten_description/urdf/tsuten_simple.urdf.xacro (robot description, xacro)
@@ -1,4 +1,5 @@
 <?xml version="1.0" encoding="UTF-8"?>
 <robot name="tsuten" xmlns:xacro="http://ros.org/wiki/xacro">
+  <xacro:include filename="$(find tsuten_description)/urdf/lidar.urdf.xacro" />
   <xacro:include filename="$(find tsuten_description)/urdf/material.urdf.xacro" />
   <xacro:include filename="$(find tsuten_description)/urdf/omni_wheel.urdf.xacro" />
@@ -54,4 +55,7 @@
       rpy="${radians(-45)} ${radians(-90)} 0" />
   </xacro:omni_wheel>
+  <xacro:lidar parent="body_link">
+    <origin xyz="-30.69e-3 283.7e-3 -164.8e-3" rpy="0 0 ${radians(90)}" />
+  </xacro:lidar>
   <gazebo reference="body_link">
     <material>

Commit message: シミュレーションの足回り制御をbase_linkに直接速度を設定するように変更

File: tsuten_description/urdf/tsuten.urdf.xacro (robot description, xacro)
@@ -3,12 +3,12 @@
   <xacro:include filename="$(find tsuten_description)/urdf/lidar.urdf.xacro" />
   <xacro:include filename="$(find tsuten_description)/urdf/material.urdf.xacro" />
-  <xacro:include filename="$(find tsuten_description)/urdf/wheel.urdf.xacro" />
-  <xacro:property name="body_mesh_path" value="$(find tsuten_description)/meshes/tsuten.stl" />
-  <xacro:property name="bumper_mesh_path" value="$(find tsuten_description)/meshes/bumper.stl" />
+  <xacro:property name="body_visual_mesh_path" value="$(find tsuten_description)/meshes/tsuten.stl" />
+  <xacro:property name="body_collision_mesh_path"
+    value="$(find tsuten_description)/meshes/tsuten_lq.stl" />
   <link name="base_link" />
   <link name="body_link">
     <visual>
       <geometry>
-        <mesh filename="${body_mesh_path}" />
+        <mesh filename="${body_visual_mesh_path}" />
       </geometry>
       <material name="Grey" />
@@ -16,5 +16,5 @@
     <collision>
       <geometry>
-        <mesh filename="${body_mesh_path}" />
+        <mesh filename="${body_collision_mesh_path}" />
       </geometry>
     </collision>
@@ -27,87 +27,18 @@
   </link>
   <joint name="body_joint" type="fixed">
-    <origin xyz="30.693e-3 3.279e-3 292.306e-3" rpy="0 0 0" />
+    <origin xyz="30.69e-3 3.279e-3 292.3e-3" rpy="0 0 0" />
     <axis xyz="0 0 1" />
     <parent link="base_link" />
     <child link="body_link" />
   </joint>
-  <link name="bumper_link">
-    <visual>
-      <geometry>
-        <mesh filename="${bumper_mesh_path}" />
-      </geometry>
-      <material name="Grey" />
-    </visual>
-    <collision name="bumper_collision">
-      <geometry name="bumper_collision">
-        <mesh filename="${bumper_mesh_path}" />
-      </geometry>
-    </collision>
-    <inertial>
-      <origin xyz="260e-3 -2.667e-3 5.00e-3" />
-      <mass value="14.607e-3" />
-      <inertia ixx="0" ixy="0" ixz="0" iyy="4.934e-4" iyz="0"
-        izz="4.974e-4" />
-    </inertial>
-  </link>
-  <joint name="bumper_joint" type="fixed">
-    <origin xyz="-290.693e-3 409.221e-3 -252.314e-3" rpy="0 0 0" />
-    <axis xyz="0 0 1" />
-    <parent link="body_link" />
-    <child link="bumper_link" />
-  </joint>
-  <xacro:wheel prefix="rf" parent="body_link">
-    <origin xyz="325.1e-3 352.5e-3 -242.3e-3" rpy="${radians(45)} ${radians(-90)} 0" />
-  </xacro:wheel>
-  <xacro:wheel prefix="lf" parent="body_link">
-    <origin xyz="-386.5e-3 352.5e-3 -242.3e-3" rpy="${radians(45)} ${radians(90)} 0" />
-  </xacro:wheel>
-  <xacro:wheel prefix="lb" parent="body_link">
-    <origin xyz="-386.5e-3 -359.1e-3 -242.3e-3" rpy="${radians(-45)} ${radians(90)} 0" />
-  </xacro:wheel>
-  <xacro:wheel prefix="rb" parent="body_link">
-    <origin xyz="325.1e-3 -359.1e-3 -242.3e-3" rpy="${radians(-45)} ${radians(-90)} 0" />
-  </xacro:wheel>
   <xacro:lidar parent="body_link">
     <origin xyz="-30.69e-3 283.7e-3 -164.8e-3" rpy="0 0 ${radians(90)}" />
   </xacro:lidar>
   <gazebo reference="body_link">
-    <material>
-      Gazebo/Grey</material>
-    <mu1 value="0.01" />
-    <mu2 value="0.01" />
-    <selfCollide value="true" />
-  </gazebo>
-  <gazebo reference="bumper_link">
-    <material>
-      Gazebo/Grey</material>
-    <mu1 value="0.01" />
-    <mu2 value="0.01" />
-    <selfCollide value="true" />
-    <!-- <sensor name="bumper_sensor" type="contact">
-      <contact>
-        <collision>bumper_collision</collision>
-      </contact>
-      <plugin name="gazebo_ros_bumper" filename="libgazebo_ros_bumper.so">
-        <alwaysOn>true</alwaysOn>
-        <updateRate>10.0</updateRate>
-        <bumperTopicName>
-          bumper</bumperTopicName>
-        <frameName>world</frameName>
-      </plugin>
-    </sensor> -->
+    <material>Gazebo/Grey</material>
+    <mu1 value="0" />
+    <mu2 value="0" />
   </gazebo>
   <gazebo>
-    <plugin name="gazebo_ros_control" filename="libgazebo_ros_control.so" />
-    <plugin name="joint_state_publisher" filename="libgazebo_ros_joint_state_publisher.so">
-      <jointName>
-        rf_wheel_joint,
-        lf_wheel_joint,
-        lb_wheel_joint,
-        rb_wheel_joint
-      </jointName>
-      <updateRate>
-        100.0</updateRate>
-    </plugin>
     <plugin name="gazebo_ros_p3d" filename="libgazebo_ros_p3d.so">
       <frameName>map</frameName>
@@ -116,4 +47,12 @@
       <updateRate>100.0</updateRate>
     </plugin>
+    <plugin name="chassis_controller" filename="libgazebo_ros_planar_move.so">
+      <commandTopic>cmd_vel</commandTopic>
+      <cmdTimeout>-1</cmdTimeout>
+      <odometryTopic>odom</odometryTopic>
+      <odometryFrame>odom</odometryFrame>
+      <odometryRate>100.0</odometryRate>
+      <robotBaseFrame>base_link</robotBaseFrame>
+    </plugin>
   </gazebo>
 </robot>

Commit message: イナーシャの設定がよくなかったので修正

File: tsuten_description/urdf/tsuten.urdf.xacro (robot description, xacro)
@@ -6,4 +6,8 @@
   <xacro:property name="body_collision_mesh_path"
     value="$(find tsuten_description)/meshes/tsuten_lq.stl" />
+  <xacro:property name="body_mass" value="30.0" />
+  <xacro:property name="body_inertia_box_x" value="800.0e-3" />
+  <xacro:property name="body_inertia_box_y" value="800.0e-3" />
+  <xacro:property name="body_inertia_box_z" value="100.0e-3" />
   <link name="base_link" />
   <link name="body_link">
@@ -20,8 +24,9 @@
     </collision>
     <inertial>
-      <origin xyz="98.435e-3 -264.408e-3 77.899e-3" />
-      <mass value="29987.685e-3" />
-      <inertia ixx="1.303e+0" ixy="1.556e-1" ixz="3.533e-2" iyy="1.465e+0" iyz="1.362e-2"
-        izz="1.212e+0" />
+      <origin xyz="-30.69e-3 -3.279e-3 -242.3e-3" />
+      <mass value="${body_mass}" />
+      <inertia ixx="${body_mass*(body_inertia_box_y**2+body_inertia_box_z**2)/12}" ixy="0" ixz="0"
+        iyy="${body_mass*(body_inertia_box_x**2+body_inertia_box_z**2)/12}" iyz="0"
+        izz="${body_mass*(body_inertia_box_x**2+body_inertia_box_y**2)/12}" />
     </inertial>
   </link>

Commit message: ポールの検出を追加

File: tsuten_description/urdf/tsuten.urdf.xacro (robot description, xacro)
@@ -38,5 +38,5 @@
   </joint>
   <xacro:lidar parent="body_link">
-    <origin xyz="-30.69e-3 283.7e-3 -164.8e-3" rpy="0 0 ${radians(90)}" />
+    <origin xyz="-30.69e-3 283.7e-3 107.7e-3" rpy="0 0 ${radians(90)}" />
   </xacro:lidar>
   <gazebo reference="body_link">

Commit message: テーブルのポール検出を台座の面の検出に変更

File: tsuten_description/urdf/tsuten.urdf.xacro (robot description, xacro)
@@ -38,5 +38,5 @@
   </joint>
   <xacro:lidar parent="body_link">
-    <origin xyz="-30.69e-3 283.7e-3 107.7e-3" rpy="0 0 ${radians(90)}" />
+    <origin xyz="-30.69e-3 283.7e-3 -164.8e-3" rpy="0 0 ${radians(90)}" />
   </xacro:lidar>
   <gazebo reference="body_link">
